File: Hardware/Rev2/Rev2.kicad_pcb (KiCad board)
At the start: 2 copper layers, 236.6 x 177.8 mm, 1058 parts, among them J1 USB_C_Receptacle_USB2.0_16P, J2 Conn_01x08, J3 Micro_SD_Card_Det1, J4 Conn_02x04_Odd_Even, SW1 SW_Push, SW2 SW_Push, U1 AW20216S, U10 AW20216S, U11 AW20216S, U12 74LS125, U13 74LS125, U14 74LS125, U15 ESP32-S3-WROOM-1, U16 USBLC6-2SC6, U17 XC6220B331MR, U2 AW20216S, U3 AW20216S, U4 AW20216S, U5 AW20216S, U6 AW20216S, U7 AW20216S, U8 AW20216S, U9 AW20216S

Commit message: hopefully final board design
Other:
- board text added: "Rev.2 / ESP32-S3 For more info: github.com/itsmevjnk/MelbourneTrainTracker Transport Pictograms, GTFS Schedule and GTFS Realtime API by the Department of Transport and Planning are licensed under CC BY 4.0."
- board text removed: "Rev.2 / ESP32-S3 For more info: github.com/itsmevjnk/MelbourneTrainTracker Transport Pictograms by the Department of Transport and Planning are licensed under CC BY 4.0."
