File: Hardware/Rev2/Rev2.kicad_pcb (KiCad board)
At the start: 2 copper layers, 251.6 x 177.8 mm, 1066 parts, among them J1 USB_C_Receptacle_USB2.0_16P, J2 Conn_01x08, J3 Micro_SD_Card_Det1, J4 Conn_02x04_Odd_Even, SW1 SW_Push, SW2 SW_Push, U1 AW20216S, U10 AW20216S, U11 AW20216S, U12 74LS125, U13 74LS125, U14 74LS125, U15 ESP32-S3-WROOM-1, U16 USBLC6-2SC6, U17 XC6220B331MR, U2 AW20216S, U3 AW20216S, U4 AW20216S, U5 AW20216S, U6 AW20216S, U7 AW20216S, U8 AW20216S, U9 AW20216S

Commit message: switch to hatched fill
Routing:
- net GND: track 581.9 -> 573.4 mm
- net L2_CS: track 343.1 -> 341.0 mm
- net MOSI_A: track 422.7 -> 420.6 mm
- net SCK_A: track 422.2 -> 421.4 mm
- net L3_CS: track 400.8 -> 400.0 mm
Other:
- board text added: "Rev.2C / ESP32-S3 For more info: github.com/itsmevjnk/MelbourneTrainTracker Transport Pictograms, GTFS Schedule and GTFS Realtime API by the Department of Transport and Planning are licensed under CC BY 4.0."
- board text removed: "Rev.2B / ESP32-S3 For more info: github.com/itsmevjnk/MelbourneTrainTracker Transport Pictograms, GTFS Schedule and GTFS Realtime API by the Department of Transport and Planning are licensed under CC BY 4.0."
