File: Hardware/Rev2/led3.kicad_sch (KiCad schematic)
At the start: 290 parts, among them U7 AW20216S, U8 AW20216S, U9 AW20216S

Commit message: rev.2c revised PCB layout, final
Parts:
- R190, R191, R192: MPN C2930231 -> C15401
Changed lines of the file:
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@@
 			)
 		)
-		(property "MPN" "C2930231"
+		(property "MPN" "C15401"
 			(at 34.29 143.51 90)
 			(effects
@@
 			)
 		)
-		(property "MPN" "C2930231"
+		(property "MPN" "C15401"
 			(at 34.29 54.61 90)
 			(effects
@@
 			)
 		)
-		(property "MPN" "C2930231"
+		(property "MPN" "C15401"
 			(at 35.56 232.41 90)
 			(effects
