File: Hardware/Rev2/led4.kicad_sch (KiCad schematic)
At the start: 131 parts, among them U10 AW20216S, U11 AW20216S

Commit message: rev.2c revised PCB layout, final
Parts:
- R196, R197: MPN C2930231 -> C15401
Changed lines of the file:
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@@
 			)
 		)
-		(property "MPN" "C2930231"
+		(property "MPN" "C15401"
 			(at 43.18 63.5 90)
 			(effects
@@
 			)
 		)
-		(property "MPN" "C2930231"
+		(property "MPN" "C15401"
 			(at 43.18 161.29 90)
 			(effects
